Commit message: code_3_29

File: src/bringup/param/robot.xacro (robot description, xacro)
@@ -32,4 +32,17 @@
     <origin xyz="0 0 0.65" />
   </joint>
+  <link name="laser">
+    <visual>
+      <geometry>
+        <cylinder length="0.05" radius="0.05" />
+      </geometry>
+      <material name="blue"/>
+    </visual>
+  </link>
+  <joint name="laser_link_joint" type="fixed">
+    <parent link="base_link" />
+    <child link="laser" />
+    <origin xyz="0.6 0 0.1" rpy="0 3.1415 3.1415" />
+  </joint>
   <xacro:macro name="ultrasound" params="number *origin">
     <link name="ultrasound${number}">
@@ -48,32 +61,32 @@
   </xacro:macro>
   <xacro:ultrasound number="0">
-      <origin xyz="0.65 0.2 0.3" rpy="1.5707 0 0"/>
+      <origin xyz="0.65 0.2 0.25" rpy="1.5707 0 0"/>
   </xacro:ultrasound>
   <xacro:ultrasound number="1">
-      <origin xyz="0.65 0 0.3" rpy="1.5707 0 0"/>
+      <origin xyz="0.65 0 0.25" rpy="1.5707 0 0"/>
   </xacro:ultrasound>
   <xacro:ultrasound number="2">
-      <origin xyz="0.65 -0.2 0.3" rpy="1.5707 0 0"/>
+      <origin xyz="0.65 -0.2 0.25" rpy="1.5707 0 0"/>
   </xacro:ultrasound>
   <xacro:ultrasound number="3">
-      <origin xyz="0.4 -0.4 0.3" rpy="0 0 -1.5707"/>
+      <origin xyz="0.5 -0.4 0.25" rpy="0 0 -1.5707"/>
   </xacro:ultrasound>
   <xacro:ultrasound number="4">
-      <origin xyz="0.3 -0.4 0.3" rpy="0 0 -1.5707"/>
+      <origin xyz="0.35 -0.4 0.25" rpy="0 0 -1.5707"/>
   </xacro:ultrasound>
   <xacro:ultrasound number="5">
-      <origin xyz="-0.65 -0.2 0.3" rpy="0 0 3.1415"/>
+      <origin xyz="-0.65 -0.2 0.25" rpy="0 0 3.1415"/>
   </xacro:ultrasound>
   <xacro:ultrasound number="6">
-      <origin xyz="-0.65 0 0.3" rpy="0 0 3.1415"/>
+      <origin xyz="-0.65 0 0.25" rpy="0 0 3.1415"/>
   </xacro:ultrasound>
   <xacro:ultrasound number="7">
-      <origin xyz="-0.65 0.2 0.3" rpy="0 0 3.1415"/>
+      <origin xyz="-0.65 0.2 0.25" rpy="0 0 3.1415"/>
   </xacro:ultrasound>
   <xacro:ultrasound number="8">
-      <origin xyz="0.3 0.4 0.3" rpy="0 0 1.5707"/>
+      <origin xyz="0.35 0.4 0.25" rpy="0 0 1.5707"/>
   </xacro:ultrasound>
   <xacro:ultrasound number="9">
-      <origin xyz="0.4 0.4 0.3" rpy="0 0 1.5707"/>
+      <origin xyz="0.5 0.4 0.25" rpy="0 0 1.5707"/>
   </xacro:ultrasound>
 </robot>

Commit message: change urdf

File: src/bringup/param/robot.xacro (robot description, xacro)
@@ -13,5 +13,5 @@
     <visual>
       <geometry>
-        <box size="1.3 0.8 0.6" />
+        <box size="1.0 0.7 0.6" />
       </geometry>
       <origin xyz="0 0 0.3"/>
@@ -43,5 +43,5 @@
     <parent link="base_link" />
     <child link="laser" />
-    <origin xyz="0.6 0 0.1" rpy="0 3.1415 3.1415" />
+    <origin xyz="0.45 0 0.1" rpy="0 3.1415 3.1415" />
   </joint>
   <xacro:macro name="ultrasound" params="number *origin">
@@ -61,32 +61,32 @@
   </xacro:macro>
   <xacro:ultrasound number="0">
-      <origin xyz="0.65 0.2 0.25" rpy="1.5707 0 0"/>
+      <origin xyz="0.5 0.2 0.25" rpy="1.5707 0 0"/>
   </xacro:ultrasound>
   <xacro:ultrasound number="1">
-      <origin xyz="0.65 0 0.25" rpy="1.5707 0 0"/>
+      <origin xyz="0.5 0 0.25" rpy="1.5707 0 0"/>
   </xacro:ultrasound>
   <xacro:ultrasound number="2">
-      <origin xyz="0.65 -0.2 0.25" rpy="1.5707 0 0"/>
+      <origin xyz="0.5 -0.2 0.25" rpy="1.5707 0 0"/>
   </xacro:ultrasound>
   <xacro:ultrasound number="3">
-      <origin xyz="0.5 -0.4 0.25" rpy="0 0 -1.5707"/>
+      <origin xyz="0.35 -0.35 0.25" rpy="0 0 -1.5707"/>
   </xacro:ultrasound>
   <xacro:ultrasound number="4">
-      <origin xyz="0.35 -0.4 0.25" rpy="0 0 -1.5707"/>
+      <origin xyz="0.2 -0.35 0.25" rpy="0 0 -1.5707"/>
   </xacro:ultrasound>
   <xacro:ultrasound number="5">
-      <origin xyz="-0.65 -0.2 0.25" rpy="0 0 3.1415"/>
+      <origin xyz="-0.5 -0.2 0.25" rpy="0 0 3.1415"/>
   </xacro:ultrasound>
   <xacro:ultrasound number="6">
-      <origin xyz="-0.65 0 0.25" rpy="0 0 3.1415"/>
+      <origin xyz="-0.5 0 0.25" rpy="0 0 3.1415"/>
   </xacro:ultrasound>
   <xacro:ultrasound number="7">
-      <origin xyz="-0.65 0.2 0.25" rpy="0 0 3.1415"/>
+      <origin xyz="-0.5 0.2 0.25" rpy="0 0 3.1415"/>
   </xacro:ultrasound>
   <xacro:ultrasound number="8">
-      <origin xyz="0.35 0.4 0.25" rpy="0 0 1.5707"/>
+      <origin xyz="0.2 0.35 0.25" rpy="0 0 1.5707"/>
   </xacro:ultrasound>
   <xacro:ultrasound number="9">
-      <origin xyz="0.5 0.4 0.25" rpy="0 0 1.5707"/>
+      <origin xyz="0.35 0.35 0.25" rpy="0 0 1.5707"/>
   </xacro:ultrasound>
 </robot>
