Commit message: connect with server

File: src/bringup/param/robot_twowheel.xacro (robot description, xacro)
@@ -7,10 +7,13 @@
       <color rgba="0 0 1 1"/>
   </material>
+  <material name="black">
+      <color rgba="0 0 0 1"/>
+  </material>
   <link name="base_link">
     <visual>
       <geometry>
-        <box size="0.8 0.55 0.7" />
+        <box size="0.85 0.60 0.7" />
       </geometry>
-      <origin xyz="-0.25 0 0.35"/>
+      <origin xyz="-0.205 0 0.35"/>
       <material name="white"/>
     </visual>
@@ -27,5 +30,31 @@
     <parent link="base_link" />
     <child link="velodyne" />
-    <origin xyz="0 0 0.725" />
+    <origin xyz="0.125 0 0.725" />
+  </joint>
+  <link name="laser">
+    <visual>
+      <geometry>
+        <cylinder length="0.05" radius="0.05" />
+      </geometry>
+      <material name="blue"/>
+    </visual>
+  </link>
+  <joint name="laser_link_joint" type="fixed">
+    <parent link="base_link" />
+    <child link="laser" />
+    <origin xyz="0.16 0 0.12" rpy="0 3.1415 0" />
+  </joint>
+  <link name="ultrasoundLaser">
+    <visual>
+      <geometry>
+        <cylinder length="0.05" radius="0.05" />
+      </geometry>
+      <material name="blue"/>
+    </visual>
+  </link>
+  <joint name="ultrasoundLaser_link_joint" type="fixed">
+    <parent link="base_link" />
+    <child link="ultrasoundLaser" />
+    <origin xyz="-0.04 0 0.725" />
   </joint>
 </robot>
